File: projects/xiao-harbor-breeze-60lm/xiao-harbor-breeze-60lm.kicad_sch (KiCad schematic)
At the start: 46 parts, among them CN1 XY122R-5.08-2P, CN2 XY122R-5.08-2P, J1 1165SDIG-07, J2 1165SDIG-07, Q1 UMW8205A, U1 BQ25185DLHR, U2 ME6210A33PG, U3 DW01A_C351410

Commit message: Drop graphics from BOM
Parts:
- G1, G2, TP1, TP2, TP3, TP4, TP5, TP6, TP7, TP8, TP9: now left out of the parts list
Changed lines of the file:
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@@
 		(unit 1)
 		(exclude_from_sim no)
-		(in_bom yes)
+		(in_bom no)
 		(on_board yes)
 		(dnp no)
@@
 		(unit 1)
 		(exclude_from_sim no)
-		(in_bom yes)
+		(in_bom no)
 		(on_board yes)
 		(dnp no)
@@
 		(unit 1)
 		(exclude_from_sim no)
-		(in_bom yes)
+		(in_bom no)
 		(on_board yes)
 		(dnp no)
@@
 		(unit 1)
 		(exclude_from_sim no)
-		(in_bom yes)
+		(in_bom no)
 		(on_board yes)
 		(dnp no)
@@
 		(unit 1)
 		(exclude_from_sim no)
-		(in_bom yes)
+		(in_bom no)
 		(on_board yes)
 		(dnp no)
@@
 		(unit 1)
 		(exclude_from_sim no)
-		(in_bom yes)
+		(in_bom no)
 		(on_board yes)
 		(dnp no)
@@
 		(unit 1)
 		(exclude_from_sim no)
-		(in_bom yes)
+		(in_bom no)
 		(on_board yes)
 		(dnp no)
@@
 		(unit 1)
 		(exclude_from_sim no)
-		(in_bom yes)
+		(in_bom no)
 		(on_board yes)
 		(dnp no)
@@
 		(unit 1)
 		(exclude_from_sim no)
-		(in_bom yes)
+		(in_bom no)
 		(on_board yes)
 		(dnp no)
@@
 		(unit 1)
 		(exclude_from_sim no)
-		(in_bom yes)
+		(in_bom no)
 		(on_board yes)
 		(dnp no)
@@
 		(unit 1)
 		(exclude_from_sim no)
-		(in_bom yes)
+		(in_bom no)
 		(on_board yes)
 		(dnp no)

Commit message: Fix GLB output; Vendor all libraries
The kicad binaries for Ubuntu 24.04 are linked against a buggy version
of OCCT. The most direct solution here was simply to upgrade to Ubuntu 25.04.

Additionally all referenced libraries are now vendored under lib/. This
ensures that there are no conflicts between the container definition and
the host.

Due to this, the entire lib/ directory is now tracked in git lfs.
Parts:
- C1, C2, C3, C4, C5, C6: footprint Capacitor_SMD:C_0805_2012Metric -> Capacitor_SMD_Vendor:C_0805_2012Metric; symbol Device:C_Small -> Device_Vendor:C_Small
- D1, D2, D3: footprint LED_SMD:LED_0603_1608Metric -> LED_SMD_Vendor:LED_0603_1608Metric; symbol Device:LED -> Device_Vendor:LED
- H1, H2, H3, H4: footprint MountingHole:MountingHole_3.2mm_M3_ISO7380_Pad -> MountingHole_Vendor:MountingHole_3.2mm_M3_ISO7380_Pad; symbol Mechanical:MountingHole_Pad -> Mechanical_Vendor:MountingHole_Pad
- JP1, JP2, JP3: footprint Jumper:SolderJumper-2_P1.3mm_Bridged_RoundedPad1.0x1.5mm -> Jumper_Vendor:SolderJumper-2_P1.3mm_Bridged_RoundedPad1.0x1.5mm
- R1, R10, R2, R3, R4, R5, R6, R7, R8, R9: footprint Resistor_SMD:R_0603_1608Metric -> Resistor_SMD_Vendor:R_0603_1608Metric; symbol Device:R_US -> Device_Vendor:R_US
- TH1: footprint Resistor_SMD:R_0603_1608Metric -> Resistor_SMD_Vendor:R_0603_1608Metric; symbol Device:Thermistor_NTC -> Device_Vendor:Thermistor_NTC
- TP1, TP2, TP3, TP4, TP5, TP6, TP7, TP8, TP9: footprint TestPoint:TestPoint_Pad_D1.5mm -> TestPoint_Vendor:TestPoint_Pad_D1.5mm; symbol Connector:TestPoint -> Connector_Vendor:TestPoint; now in the parts list

Commit message: Add zip-tie PCB documentation
Documents the purpose of the PCB cutout regions. Intended for users to
pass a zip-tie through and around to secure the XIAO development kit.
Parts:
- JP1, JP2, JP3: symbol Jumper:SolderJumper_2_Bridged -> Jumper_Vendor:SolderJumper_2_Bridged
Changed lines of the file:
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@@
 	)
 	(symbol
-		(lib_id "Jumper:SolderJumper_2_Bridged")
+		(lib_id "Jumper_Vendor:SolderJumper_2_Bridged")
 		(at 199.39 63.5 90)
 		(unit 1)
@@
 	)
 	(symbol
-		(lib_id "Jumper:SolderJumper_2_Bridged")
+		(lib_id "Jumper_Vendor:SolderJumper_2_Bridged")
 		(at 189.23 63.5 90)
 		(unit 1)
@@
 	)
 	(symbol
-		(lib_id "Jumper:SolderJumper_2_Bridged")
+		(lib_id "Jumper_Vendor:SolderJumper_2_Bridged")
 		(at 179.07 63.5 90)
 		(unit 1)
